Commit message: achieved slam

File: urdf/beer_bot.urdf.xacro (robot description, xacro)
@@ -7,4 +7,13 @@
   <xacro:property name="wheel_width" value="0.025"/>   <!-- Estimated wheel thickness -->
   <xacro:property name="lidar_height" value="0.175"/>   <!-- 200mm above axle -->
+<!-- === Base Footprint === -->
+  <link name="base_footprint">
+    <visual>
+      <geometry>
+        <cylinder radius="0.05" length="0.05"/>
+      </geometry>
+      <material name="blue"><color rgba="0 0 1 1"/></material>
+    </visual>
+  </link>
   <!-- === Base Link === -->
   <link name="base_link">
@@ -22,10 +31,10 @@
       </geometry>
     </collision>
-    <inertial>
+    <!-- <inertial>
       <mass value="5.0"/>
       <origin xyz="0 0 0" rpy="0 0 0"/>
       <inertia ixx="0.1" iyy="0.1" izz="0.1"
                ixy="0.0" ixz="0.0" iyz="0.0"/>
-    </inertial>
+    </inertial> -->
   </link>
   <!-- === Wheel Macro === -->
@@ -76,3 +85,8 @@
     <origin xyz="0.007 0 ${lidar_height}" rpy="0 0 0"/>
   </joint>
+    <joint name="base_joint" type="fixed">
+    <parent link="base_link"/>
+    <child link="base_footprint"/>
+    <origin xyz="0.0 0 -${wheel_radius}" rpy="0 0 0"/>
+  </joint>
 </robot>
